File: hardware/project-stemmaqt-AS7341.kicad_pcb (KiCad board)
At the start: 4 copper layers, 25.4 x 17.8 mm, 23 parts, among them J1 SM04B-SRSS-TB(LF)(SN), J2 SM04B-SRSS-TB(LF)(SN), J3 Conn_01x03_Male, Q1 Q_PMOS_GSD, U1 DS2482S-100+

Commit message: First placement
Parts:
- removed JP2: AD1, Jumper:SolderJumper-2_P1.3mm_Open_RoundedPad1.0x1.5mm
- removed JP3: SPU, Jumper:SolderJumper-2_P1.3mm_Open_RoundedPad1.0x1.5mm
- removed Q1: Q_PMOS_GSD, Package_TO_SOT_SMD:SOT-23
- removed R5: 10k, Resistor_SMD:R_0603_1608Metric
- removed R6: SPU, Resistor_SMD:R_0603_1608Metric
- added C3: 0.1uF, Capacitor_SMD:C_0603_1608Metric, F.Cu at (49.1, 63.6)
- added U2: AS7341-DLGT, AS7341-DLGT:PSON80P310X200X110-8N, F.Cu at (51.7, 63.6)
- C1: value 100nF -> 1uF; footprint Capacitor_SMD:C_0603_1608Metric -> Capacitor_SMD:C_0805_2012Metric
- C2: value 10uF -> 1uF; footprint Capacitor_SMD:C_1210_3225Metric -> Capacitor_SMD:C_0805_2012Metric
- J3: value Conn_01x03_Male -> SM04B-SRSS-TB(LF)(SN); footprint Connector_PinHeader_2.54mm:PinHeader_1x03_P2.54mm_Vertical -> SM04B-SRSS-TB(LF)(SN):JST_SM04B-SRSS-TB(LF)(SN)
- JP1: value AD0 -> SolderJumper_3_Bridged12; footprint Jumper:SolderJumper-2_P1.3mm_Open_RoundedPad1.0x1.5mm -> Jumper:SolderJumper-3_P1.3mm_Bridged12_RoundedPad1.0x1.5mm
- R1, R2, R4: value 10k -> PU
- R3: value 10k -> ?
- U1: value DS2482S-100+ -> TPS7A0218PDBVR; footprint DS2482S-100:SOIC127P600X175-8N -> TPS7A0233PDBVR:SOT95P280X145-5N
- moved C2 14.1 mm to (49.9, 57.3)
- moved R1 9.36 mm to (45.3, 64.4), turned to 180 degrees
- moved C1 8.96 mm to (42.5, 57.3)
- moved R4 8.39 mm to (45.3, 61.3), turned to 180 degrees
- moved R2 7.33 mm to (45.3, 62.9), turned to 180 degrees
- moved U1 6.84 mm to (46.4, 57.3), turned to 0 degrees
- moved JP1 3.70 mm to (55.2, 57.3), turned to 90 degrees
- moved J3 2.62 mm to (45.7, 67.4), turned to 0 degrees
- moved D1 0.76 mm to (55.8, 70.2)
- moved R3 0.76 mm to (54.0, 70.2)
Connections:
- C2 pad 1: VCC -> +1V8
- J3 pad 1: VCC -> /EN
- J3 pad 2: /1WIRE -> /GPIO
- J3 pad 3: GND -> /INT
- JP1 pad 1: VCC -> /EN
- R1 pad 1: Net-(JP1-Pad2) -> VCC
- R1 pad 2: GND -> /INT
- R2 pad 1: Net-(JP2-Pad2) -> VCC
- R2 pad 2: GND -> /SCL
- R4 pad 2: /SCL -> /SDA
- U1 pad 2: /1WIRE -> GND
- U1 pad 3: GND -> Net-(JP1-Pad2)
- U1 pad 4: /SCL -> (no net)
- U1 pad 5: /SDA -> +1V8
Routing:
- net /1WIRE: track 32.3 -> 0.00 mm
- net /SDA: track 24.9 -> 0.00 mm
- net /SCL: track 19.1 -> 0.00 mm
- net Net-(JP2-Pad2): track 13.5 -> 0.00 mm, vias 2 -> 0
- net Net-(JP1-Pad2): track 12.3 -> 0.00 mm
- net VCC: track 14.9 -> 3.50 mm, vias 9 -> 3
- net /PCTLZ: track 7.27 -> 0.00 mm, vias 2 -> 0
- net GND: track 15.9 -> 9.34 mm, vias 11 -> 7
- net Net-(JP3-Pad1): track 5.66 -> 0.00 mm
- net Net-(Q1-Pad2): track 1.64 -> 0.00 mm
Other:
- board text added: "Stemma AS7341"
- board text removed: "1W"
- board text removed: "GND"
- board text removed: "Stemma OneWire"
- board text removed: "VCC"

Commit message: Routing done
Routing:
- net /SCL: track 0.00 -> 24.2 mm
- net /SDA: track 0.00 -> 23.9 mm
- net /EN: track 0.00 -> 22.5 mm, vias 0 -> 2
- net /GPIO: track 0.00 -> 18.9 mm, vias 0 -> 2
- net /INT: track 0.00 -> 13.5 mm, vias 0 -> 3
- net Net-(JP1-Pad2): track 0.00 -> 10.5 mm, vias 0 -> 2
- net +1V8: track 0.00 -> 9.75 mm, vias 0 -> 2
- net GND: track 9.34 -> 16.4 mm, vias 7 -> 15
- net VCC: track 3.50 -> 8.15 mm, vias 3 -> 8
- added copper zone on F.Cu, net +1V8
- added copper zone on F.Cu, net GND
- added copper zone on F.Cu, net VCC
